File: hardware/gMeter-mlf.sch (KiCad schematic (older format))
At the start: 37 parts, among them IC1 ATMEGA88P, P4 USB, P5 ISP, Q1 BC847C, X1 12MHz

Commit message: Various misc corrections. Version bumped to v1.1.
Parts:
- R10, R11, R12, R13, R14: value 470 -> 1K
- R15, R16: value 470 -> 3K9
- R9: value 470 -> 1K5
Changed lines of the file:
@@
 LIBS:valves
 LIBS:npn-bce
-LIBS:tMeter-mlf-cache
-EELAYER 24 0
+LIBS:gMeter-mlf-cache
+EELAYER 27 0
 EELAYER END
 $Descr A4 11693 8268
 encoding utf-8
 Sheet 1 1
-Title "G9X USB Programmer"
-Date "1 jun 2013"
+Title "gMeter-MLF"
+Date "27 jun 2013"
 Rev "1.1"
 Comp ""
@@
 P 6550 5150
 F 0 "R16" V 6630 5150 50  0000 C CNN
-F 1 "470" V 6550 5150 50  0000 C CNN
+F 1 "3K9" V 6550 5150 50  0000 C CNN
 F 2 "" H 6550 5150 60  0001 C CNN
 F 3 "" H 6550 5150 60  0001 C CNN
@@
 P 6550 4850
 F 0 "R15" V 6630 4850 50  0000 C CNN
-F 1 "470" V 6550 4850 50  0000 C CNN
+F 1 "3K9" V 6550 4850 50  0000 C CNN
 F 2 "" H 6550 4850 60  0001 C CNN
 F 3 "" H 6550 4850 60  0001 C CNN
@@
 P 6550 4550
 F 0 "R14" V 6630 4550 50  0000 C CNN
-F 1 "470" V 6550 4550 50  0000 C CNN
+F 1 "1K" V 6550 4550 50  0000 C CNN
 F 2 "" H 6550 4550 60  0001 C CNN
 F 3 "" H 6550 4550 60  0001 C CNN
@@
 P 6550 4250
 F 0 "R13" V 6630 4250 50  0000 C CNN
-F 1 "470" V 6550 4250 50  0000 C CNN
+F 1 "1K" V 6550 4250 50  0000 C CNN
 F 2 "" H 6550 4250 60  0001 C CNN
 F 3 "" H 6550 4250 60  0001 C CNN
@@
 P 6550 3950
 F 0 "R12" V 6630 3950 50  0000 C CNN
-F 1 "470" V 6550 3950 50  0000 C CNN
+F 1 "1K" V 6550 3950 50  0000 C CNN
 F 2 "" H 6550 3950 60  0001 C CNN
 F 3 "" H 6550 3950 60  0001 C CNN
@@
 P 6550 3650
 F 0 "R11" V 6630 3650 50  0000 C CNN
-F 1 "470" V 6550 3650 50  0000 C CNN
+F 1 "1K" V 6550 3650 50  0000 C CNN
 F 2 "" H 6550 3650 60  0001 C CNN
 F 3 "" H 6550 3650 60  0001 C CNN
@@
 P 6550 3350
 F 0 "R10" V 6630 3350 50  0000 C CNN
-F 1 "470" V 6550 3350 50  0000 C CNN
+F 1 "1K" V 6550 3350 50  0000 C CNN
 F 2 "" H 6550 3350 60  0001 C CNN
 F 3 "" H 6550 3350 60  0001 C CNN
@@
 P 6550 3050
 F 0 "R9" V 6630 3050 50  0000 C CNN
-F 1 "470" V 6550 3050 50  0000 C CNN
+F 1 "1K5" V 6550 3050 50  0000 C CNN
 F 2 "" H 6550 3050 60  0001 C CNN
 F 3 "" H 6550 3050 60  0001 C CNN

Commit message: + New firmware-mlf folder for gMeter-MLF version, though no changes   except fuse settings at this time + Reduced some via sizes on MLF board + Moved a couple component value texts on MLF board + Added two MLF version first build wiki images
Parts:
- IC1: symbol ATMEGA48P -> ATMEGA88P
Connections:
- net GND: now also IC1.0 (GND)
Changed lines of the file:
@@
 LIBS:npn-bce
 LIBS:gMeter-mlf-cache
-EELAYER 27 0
+EELAYER 24 0
 EELAYER END
 $Descr A4 11693 8268
@@
 	4050 3700 4050 3850
 Wire Wire Line
-	3950 6600 4150 6600
+	3950 6600 5000 6600
 Connection ~ 4050 6600
 Wire Wire Line
@@
 $EndComp
 $Comp
-L ATMEGA48P IC1
+L ATMEGA88P IC1
 U 1 1 4ECC4939
 P 4050 5100
@@
 	1    0    0    -1
 $EndComp
+Wire Wire Line
+	5000 6600 5000 6050
+Connection ~ 4150 6600
 $EndSCHEMATC
